File: Board/ESP12_Receipt_Printer.brd (EAGLE design)
At the start: 80 x 35 mm, 19 parts, among them CON1 BARREL_JACK_3PINPJ-102A_2MM_H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, U1 ESP-12E, U2 AMS1117

Commit message: Updated to correct board files
Parts:
- added R8: (no value), DR:M0805
- added SW1: SW_TOGGLE_6PIN_DPDT, DR:BTN_6PIN
- moved C1 19.5 mm to (69.5, 31.0), turned to 90 degrees
- moved C2 16.6 mm to (61.1, 31.1)
- moved U$1 15.5 mm to (67.3, 29.2), turned to 180 degrees
Connections:
- removed net +9V: C1.1, CON1.1, R3.2, U$1.1
- new net +9VSW: C1.1, R3.2, SW1.P$3, SW1.P$4, U$1.1
- new net +9V_SW: CON1.1, SW1.P$2, SW1.P$5
- new net N$7: R8.2, U1.10
- net +3V3: now also U1.3
- net GND: now also R8.1
Routing:
- net +9V: track 91.3 -> 0.00 mm, vias 2 -> 0
- net +9VSW: track 0.00 -> 91.1 mm, vias 0 -> 2
- net +9V_SW: track 0.00 -> 23.4 mm
- net +3V3: track 47.3 -> 62.3 mm
- net +5V: track 51.9 -> 43.5 mm
- net N$7: track 0.00 -> 4.45 mm
Changed lines of the file:
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@@
 <layer number="23" name="tOrigins" color="15" fill="1" visible="yes" active="yes"/>
 <layer number="24" name="bOrigins" color="15" fill="1" visible="yes" active="yes"/>
-<layer number="25" name="tNames" color="7" fill="1" visible="yes" active="yes"/>
+<layer number="25" name="tNames" color="7" fill="1" visible="no" active="yes"/>
 <layer number="26" name="bNames" color="7" fill="1" visible="yes" active="yes"/>
-<layer number="27" name="tValues" color="7" fill="1" visible="yes" active="yes"/>
-<layer number="28" name="bValues" color="7" fill="1" visible="yes" active="yes"/>
+<layer number="27" name="tValues" color="7" fill="1" visible="no" active="yes"/>
+<layer number="28" name="bValues" color="7" fill="1" visible="no" active="yes"/>
 <layer number="29" name="tStop" color="7" fill="3" visible="no" active="yes"/>
 <layer number="30" name="bStop" color="7" fill="6" visible="no" active="yes"/>
@@
 <element name="BTN1" library="DR" package="SMD-2-SWITCH" value="FSMSM_SWITCH_6X3.6" x="24.13" y="6.35" smashed="yes" rot="R180"/>
 <element name="BTN2" library="DR" package="SMD-2-SWITCH" value="FSMSM_SWITCH_6X3.6" x="10.16" y="6.35" smashed="yes" rot="R180"/>
-<element name="C1" library="DR" package="C0805" value="" x="76.2" y="12.7" smashed="yes" rot="R270">
-<attribute name="NAME" x="77.47" y="13.97" size="1.27" layer="25" rot="R270"/>
-<attribute name="VALUE" x="73.66" y="13.97" size="1.27" layer="27" rot="R270"/>
-</element>
-<element name="C2" library="DR" package="C0805" value="" x="76.2" y="24.13" smashed="yes" rot="R90">
-<attribute name="NAME" x="74.93" y="22.86" size="1.27" layer="25" rot="R90"/>
-<attribute name="VALUE" x="78.74" y="22.86" size="1.27" layer="27" rot="R90"/>
+<element name="C1" library="DR" package="C0805" value="" x="69.469" y="30.988" smashed="yes" rot="R90">
+<attribute name="NAME" x="68.199" y="29.718" size="1.27" layer="25" rot="R90"/>
+<attribute name="VALUE" x="72.009" y="29.718" size="1.27" layer="27" rot="R90"/>
+</element>
+<element name="C2" library="DR" package="C0805" value="" x="61.087" y="31.115" smashed="yes" rot="R90">
+<attribute name="NAME" x="59.817" y="29.845" size="1.27" layer="25" rot="R90"/>
+<attribute name="VALUE" x="63.627" y="29.845" size="1.27" layer="27" rot="R90"/>
 </element>
 <element name="C3" library="DR" package="C0805" value="" x="31.75" y="8.89" smashed="yes" rot="R270">
@@
 <attribute name="VALUE" x="2.54" y="26.67" size="1.27" layer="27" rot="R270"/>
 </element>
-<element name="U$1" library="DR" package="TO252-3" value="7805" x="76.2" y="16.51" smashed="yes" rot="R90"/>
+<element name="U$1" library="DR" package="TO252-3" value="7805" x="67.31" y="29.21" smashed="yes" rot="R180"/>
 <element name="JP2" library="pinhead" library_urn="urn:adsk.eagle:library:325" package="1X02/90" package3d_urn="urn:adsk.eagle:package:22437/2" value="" x="57.15" y="11.43" smashed="yes" rot="MR180">
 <attribute name="NAME" x="53.975" y="15.24" size="1.27" layer="26" ratio="10" rot="MR270"/>
@@
 <attribute name="VALUE" x="31.75" y="19.05" size="1.27" layer="27" rot="R180"/>
 </element>
+<element name="R8" library="DR" package="M0805" value="" x="29.21" y="12.7" smashed="yes" rot="R90">
+<attribute name="NAME" x="27.94" y="11.43" size="1.27" layer="25" rot="R90"/>
+<attribute name="VALUE" x="31.75" y="11.43" size="1.27" layer="27" rot="R90"/>
+</element>
+<element name="SW1" library="DR" package="BTN_6PIN" value="SW_TOGGLE_6PIN_DPDT" x="76.2" y="20.32" smashed="yes" rot="R180"/>
 </elements>
 <signals>
@@
 <via x="31.242" y="22.098" extent="1-16" drill="0.9" diameter="1.3"/>
 <wire x1="31.242" y1="28.448" x2="31.242" y2="22.098" width="0.6096" layer="16"/>
+<contactref element="R8" pad="1"/>
 </signal>
 <signal name="N$1">
@@
 <wire x1="5.08" y1="12.7" x2="5.273" y2="12.507" width="0.8128" layer="1"/>
 <wire x1="5.273" y1="12.507" x2="5.461" y2="12.507" width="0.8128" layer="1"/>
-</signal>
-<signal name="+9V">
-<contactref element="C1" pad="1"/>
+<contactref element="U1" pad="3"/>
+<wire x1="8.79" y1="12.7" x2="10.16" y2="12.7" width="0.6096" layer="1"/>
+<wire x1="12.7" y1="15.24" x2="12.7" y2="20.32" width="0.6096" layer="1"/>
+<wire x1="12.7" y1="20.32" x2="10.32" y2="22.7" width="0.6096" layer="1"/>
+<wire x1="10.32" y1="22.7" x2="8.79" y2="22.7" width="0.6096" layer="1"/>
+<wire x1="10.16" y1="12.7" x2="12.7" y2="15.24" width="0.6096" layer="1"/>
+</signal>
+<signal name="+9V_SW">
 <contactref element="CON1" pad="1"/>
-<contactref element="R3" pad="2"/>
-<contactref element="U$1" pad="1"/>
 <wire x1="63.5" y1="7.62" x2="63.5" y2="8.89" width="1.27" layer="1"/>
-<wire x1="63.5" y1="8.89" x2="67.31" y2="12.7" width="1.27" layer="1"/>
-<wire x1="73.66" y1="12.7" x2="76.2" y2="15.24" width="1.27" layer="1"/>
-<wire x1="76.2" y1="15.24" x2="76.2" y2="16.51" width="1.27" layer="1"/>
-<wire x1="67.31" y1="12.7" x2="73.66" y2="12.7" width="1.27" layer="1"/>
-<via x="4.953" y="18.542" extent="1-16" drill="0.9" diameter="1.3"/>
-<wire x1="5.08" y1="20.64" x2="5.08" y2="18.669" width="0.8128" layer="1"/>
-<wire x1="5.08" y1="18.669" x2="4.953" y2="18.542" width="0.8128" layer="1"/>
-<via x="62.103" y="10.922" extent="1-16" drill="0.9" diameter="1.3"/>
-<wire x1="62.103" y1="10.922" x2="63.5" y2="9.525" width="0.6096" layer="1"/>
+<wire x1="63.5" y1="8.89" x2="66.675" y2="12.065" width="1.27" layer="1"/>
 <wire x1="63.5" y1="9.525" x2="63.5" y2="7.62" width="0.6096" layer="1"/>
-<wire x1="4.953" y1="18.542" x2="61.468" y2="18.542" width="0.6096" layer="16"/>
-<wire x1="61.468" y1="18.542" x2="62.23" y2="17.78" width="0.6096" layer="16"/>
-<wire x1="62.23" y1="17.78" x2="62.23" y2="11.049" width="0.6096" layer="16"/>
-<wire x1="62.23" y1="11.049" x2="62.103" y2="10.922" width="0.6096" layer="16"/>
-<wire x1="76.2" y1="13.65" x2="76.2" y2="16.51" width="1.27" layer="1"/>
+<contactref element="SW1" pad="P$5"/>
+<contactref element="SW1" pad="P$2"/>
+<wire x1="74.1" y1="12.065" x2="66.675" y2="12.065" width="1.016" layer="1"/>
+<wire x1="74.1" y1="16.12" x2="74.1" y2="12.065" width="1.016" layer="1"/>
+<wire x1="74.1" y1="16.12" x2="74.1" y2="20.22" width="1.016" layer="1"/>
+<wire x1="74.1" y1="20.22" x2="74.2" y2="20.32" width="1.016" layer="1"/>
 </signal>
 <signal name="+5V">
@@
 <contactref element="U$1" pad="3"/>
 <contactref element="JP2" pad="1"/>
-<wire x1="76.2" y1="21.07" x2="76.2" y2="23.18" width="1.27" layer="1"/>
-<wire x1="76.2" y1="23.18" x2="73.34" y2="23.18" width="1.27" layer="1"/>
-<wire x1="71.12" y1="25.4" x2="63.5" y2="25.4" width="1.27" layer="1"/>
-<wire x1="63.5" y1="25.4" x2="55.88" y2="17.78" width="1.27" layer="1"/>
-<wire x1="55.88" y1="17.78" x2="55.88" y2="15.24" width="1.27" layer="1"/>
-<wire x1="73.34" y1="23.18" x2="71.12" y2="25.4" width="1.27" layer="1"/>
+<wire x1="55.88" y1="24.13" x2="55.88" y2="15.24" width="1.27" layer="1"/>
 <wire x1="55.88" y1="15.24" x2="55.88" y2="12.7" width="0.8128" layer="1"/>
 <wire x1="55.88" y1="12.7" x2="49.53" y2="6.35" width="0.8128" layer="1"/>
 <wire x1="49.53" y1="6.35" x2="39.37" y2="6.35" width="0.8128" layer="1"/>
 <wire x1="39.37" y1="6.35" x2="39.37" y2="5.5" width="0.8128" layer="1"/>
+<wire x1="62.75" y1="29.21" x2="61.552528125" y2="29.21" width="1.016" layer="1"/>
+<wire x1="61.552528125" y1="29.21" x2="61.087" y2="30.165" width="1.016" layer="1"/>
+<wire x1="61.087" y1="30.165" x2="58.570621875" y2="30.165" width="1.016" layer="1"/>
+<wire x1="58.570621875" y1="30.165" x2="58.195496875" y2="26.445496875" width="1.016" layer="1"/>
+<wire x1="55.88" y1="24.13" x2="58.195496875" y2="26.445496875" width="1.016" layer="1"/>
 </signal>
 <signal name="N$3">
@@
 <wire x1="48.26" y1="15.24" x2="48.26" y2="18.1" width="0.8128" layer="1"/>
 </signal>
+<signal name="N$7">
+<contactref element="R8" pad="2"/>
+<contactref element="U1" pad="10"/>
+<wire x1="25.19" y1="14.7" x2="27.21" y2="14.7" width="0.6096" layer="1"/>
+<wire x1="28.26" y1="13.65" x2="29.21" y2="13.65" width="0.6096" layer="1"/>
+<wire x1="27.21" y1="14.7" x2="28.26" y2="13.65" width="0.6096" layer="1"/>
+</signal>
+<signal name="+9VSW">
+<contactref element="C1" pad="1"/>
+<contactref element="R3" pad="2"/>
+<contactref element="U$1" pad="1"/>
+<wire x1="69.469" y1="30.038" x2="68.9" y2="29.21" width="1.27" layer="1"/>
+<wire x1="68.9" y1="29.21" x2="67.31" y2="29.21" width="1.27" layer="1"/>
+<contactref element="SW1" pad="P$4"/>
+<contactref element="SW1" pad="P$3"/>
+<via x="5.08" y="16.51" extent="1-16" drill="0.9" diameter="1.3"/>
+<via x="66.04" y="16.51" extent="1-16" drill="0.9" diameter="1.3"/>
+<wire x1="5.08" y1="16.51" x2="43.18" y2="16.51" width="0.6096" layer="16"/>
+<wire x1="43.18" y1="16.51" x2="45.72" y2="19.05" width="0.6096" layer="16"/>
+<wire x1="45.72" y1="19.05" x2="63.5" y2="19.05" width="0.6096" layer="16"/>
+<wire x1="63.5" y1="19.05" x2="66.04" y2="16.51" width="0.6096" layer="16"/>
+<wire x1="5.08" y1="16.51" x2="5.08" y2="20.64" width="0.6096" layer="1"/>
+<wire x1="72.2" y1="20.32" x2="72.2" y2="27.307" width="1.016" layer="1"/>
+<wire x1="72.2" y1="27.307" x2="69.469" y2="30.038" width="1.016" layer="1"/>
+<wire x1="72.1" y1="16.12" x2="72.1" y2="20.22" width="1.016" layer="1"/>
+<wire x1="72.1" y1="20.22" x2="72.2" y2="20.32" width="1.016" layer="1"/>
+<wire x1="72.1" y1="16.12" x2="66.43" y2="16.12" width="1.016" layer="1"/>
+<wire x1="66.43" y1="16.12" x2="66.04" y2="16.51" width="1.016" layer="1"/>
+</signal>
 </signals>
