File: Board/ESP12_Receipt_Printer.sch (EAGLE design)
At the start: 19 parts, among them CON1 BARREL_JACK_3PINPJ-102A_2MM_H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, U1 ESP-12E, U2 AMS1117

Commit message: Updated to correct board files
Parts:
- added R8: (no value), DR:R-US_M0805
- added SW1: SW_TOGGLE_6PIN_DPDT, DR:SW_TOGGLE_6PIN_DPDT
Connections:
- removed net +9V: C1.1, CON1.TIP, R3.2, U$1.VIN
- new net +9VSW: C1.1, R3.2, SW1.NO_1, SW1.NO_2, U$1.VIN
- new net +9V_SW: CON1.TIP, SW1.C_1, SW1.C_2
- new net N$7: R8.2, U1.GPIO15
- net +3V3: now also U1.CH_PD\
- net GND: now also R8.1
Other:
- moved on the sheet: R2
Changed lines of the file:
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@@
 <part name="R6" library="DR" deviceset="R-US_" device="M0805"/>
 <part name="R7" library="DR" deviceset="R-US_" device="M0805"/>
+<part name="R8" library="DR" deviceset="R-US_" device="M0805"/>
+<part name="SW1" library="DR" deviceset="SW_TOGGLE_6PIN_DPDT" device=""/>
+<part name="SUPPLY3" library="supply2" library_urn="urn:adsk.eagle:library:372" deviceset="+9V" device=""/>
 </parts>
 <sheets>
@@
 <attribute name="VALUE" x="83.82" y="38.1" size="1.778" layer="96"/>
 </instance>
-<instance part="R2" gate="G$1" x="71.12" y="50.8" smashed="yes" rot="R90">
-<attribute name="NAME" x="69.6214" y="46.99" size="1.778" layer="95" rot="R90"/>
-<attribute name="VALUE" x="74.422" y="46.99" size="1.778" layer="96" rot="R90"/>
+<instance part="R2" gate="G$1" x="71.12" y="58.42" smashed="yes" rot="R90">
+<attribute name="NAME" x="69.6214" y="54.61" size="1.778" layer="95" rot="R90"/>
+<attribute name="VALUE" x="74.422" y="54.61" size="1.778" layer="96" rot="R90"/>
 </instance>
 <instance part="+3V1" gate="G$1" x="20.32" y="73.66" smashed="yes">
@@
 <attribute name="VALUE" x="122.555" y="92.075" size="1.778" layer="96"/>
 </instance>
-<instance part="SUPPLY2" gate="G$1" x="5.08" y="99.06" smashed="yes">
-<attribute name="VALUE" x="3.175" y="102.235" size="1.778" layer="96"/>
-</instance>
+<instance part="SUPPLY2" gate="G$1" x="5.08" y="99.06" smashed="yes"/>
 <instance part="GND6" gate="1" x="119.38" y="76.2" smashed="yes">
 <attribute name="VALUE" x="116.84" y="73.66" size="1.778" layer="96"/>
@@
 <attribute name="NAME" x="77.47" y="36.6014" size="1.778" layer="95" rot="R180"/>
 <attribute name="VALUE" x="77.47" y="41.402" size="1.778" layer="96" rot="R180"/>
+</instance>
+<instance part="R8" gate="G$1" x="66.04" y="30.48" smashed="yes" rot="R90">
+<attribute name="NAME" x="64.5414" y="26.67" size="1.778" layer="95" rot="R90"/>
+<attribute name="VALUE" x="69.342" y="26.67" size="1.778" layer="96" rot="R90"/>
+</instance>
+<instance part="SW1" gate="G$1" x="137.16" y="60.96" smashed="yes">
+<attribute name="NAME" x="142.24" y="46.99" size="1.778" layer="95"/>
+</instance>
+<instance part="SUPPLY3" gate="G$1" x="129.54" y="66.04" smashed="yes">
+<attribute name="VALUE" x="127.635" y="69.215" size="1.778" layer="96"/>
 </instance>
 </instances>
@@
 <pinref part="U1" gate="G$1" pin="GND"/>
 <pinref part="GND3" gate="1" pin="GND"/>
+<wire x1="60.96" y1="43.18" x2="63.5" y2="43.18" width="0.1524" layer="91"/>
+<junction x="60.96" y="43.18"/>
+<wire x1="63.5" y1="43.18" x2="63.5" y2="25.4" width="0.1524" layer="91"/>
+<pinref part="R8" gate="G$1" pin="1"/>
+<wire x1="63.5" y1="25.4" x2="66.04" y2="25.4" width="0.1524" layer="91"/>
 </segment>
 <segment>
@@
 <pinref part="R2" gate="G$1" pin="1"/>
 <pinref part="U1" gate="G$1" pin="GPIO0/FLASH"/>
-<wire x1="71.12" y1="45.72" x2="60.96" y2="50.8" width="0.1524" layer="91"/>
-<junction x="71.12" y="45.72"/>
+<wire x1="71.12" y1="53.34" x2="60.96" y2="50.8" width="0.1524" layer="91"/>
+<junction x="71.12" y="53.34"/>
+<wire x1="71.12" y1="53.34" x2="71.12" y2="45.72" width="0.1524" layer="91"/>
 </segment>
 </net>
@@
 <pinref part="R2" gate="G$1" pin="2"/>
 <pinref part="+3V2" gate="G$1" pin="+3V3"/>
-<wire x1="71.12" y1="66.04" x2="71.12" y2="55.88" width="0.1524" layer="91"/>
+<wire x1="71.12" y1="66.04" x2="71.12" y2="63.5" width="0.1524" layer="91"/>
 </segment>
 <segment>
 <pinref part="U1" gate="G$1" pin="VCC"/>
 <pinref part="+3V3" gate="G$1" pin="+3V3"/>
-<wire x1="22.86" y1="43.18" x2="2.54" y2="43.18" width="0.1524" layer="91"/>
+<wire x1="22.86" y1="43.18" x2="20.32" y2="43.18" width="0.1524" layer="91"/>
+<pinref part="U1" gate="G$1" pin="CH_PD\"/>
+<wire x1="20.32" y1="43.18" x2="2.54" y2="43.18" width="0.1524" layer="91"/>
+<wire x1="22.86" y1="55.88" x2="20.32" y2="55.88" width="0.1524" layer="91"/>
+<wire x1="20.32" y1="55.88" x2="20.32" y2="43.18" width="0.1524" layer="91"/>
+<junction x="20.32" y="43.18"/>
 </segment>
 <segment>
@@
 </segment>
 </net>
-<net name="+9V" class="0">
-<segment>
-<pinref part="C1" gate="G$1" pin="1"/>
-<wire x1="5.08" y1="96.52" x2="5.08" y2="93.98" width="0.1524" layer="91"/>
-<pinref part="SUPPLY2" gate="G$1" pin="+9V"/>
-<junction x="5.08" y="96.52"/>
-<pinref part="R3" gate="G$1" pin="2"/>
-<wire x1="5.08" y1="96.52" x2="-7.62" y2="96.52" width="0.1524" layer="91"/>
-<pinref part="U$1" gate="G$1" pin="VIN"/>
-</segment>
+<net name="+9V_SW" class="0">
 <segment>
 <pinref part="CON1" gate="G$1" pin="TIP"/>
@@
 <wire x1="119.38" y1="83.82" x2="124.46" y2="83.82" width="0.1524" layer="91"/>
 <wire x1="124.46" y1="83.82" x2="124.46" y2="86.36" width="0.1524" layer="91"/>
+</segment>
+<segment>
+<pinref part="SW1" gate="G$1" pin="C_2"/>
+<pinref part="SW1" gate="G$1" pin="C_1"/>
+<wire x1="137.16" y1="54.61" x2="137.16" y2="60.96" width="0.1524" layer="91"/>
+<wire x1="137.16" y1="60.96" x2="129.54" y2="60.96" width="0.1524" layer="91"/>
+<junction x="137.16" y="60.96"/>
+<wire x1="129.54" y1="60.96" x2="129.54" y2="63.5" width="0.1524" layer="91"/>
+<pinref part="SUPPLY3" gate="G$1" pin="+9V"/>
 </segment>
 </net>
@@
 <segment>
 <pinref part="U1" gate="G$1" pin="GPIO2"/>
-<wire x1="60.96" y1="48.26" x2="63.5" y2="48.26" width="0.1524" layer="91"/>
-<wire x1="63.5" y1="48.26" x2="63.5" y2="43.18" width="0.1524" layer="91"/>
-<wire x1="63.5" y1="43.18" x2="68.58" y2="43.18" width="0.1524" layer="91"/>
+<wire x1="60.96" y1="48.26" x2="68.58" y2="48.26" width="0.1524" layer="91"/>
 <pinref part="R7" gate="G$1" pin="2"/>
-<wire x1="68.58" y1="43.18" x2="68.58" y2="38.1" width="0.1524" layer="91"/>
+<wire x1="68.58" y1="48.26" x2="68.58" y2="38.1" width="0.1524" layer="91"/>
 </segment>
 </net>
@@
 </segment>
 </net>
+<net name="N$7" class="0">
+<segment>
+<pinref part="R8" gate="G$1" pin="2"/>
+<wire x1="66.04" y1="35.56" x2="66.04" y2="45.72" width="0.1524" layer="91"/>
+<pinref part="U1" gate="G$1" pin="GPIO15"/>
+<wire x1="66.04" y1="45.72" x2="60.96" y2="45.72" width="0.1524" layer="91"/>
+</segment>
+</net>
+<net name="+9VSW" class="0">
+<segment>
+<pinref part="C1" gate="G$1" pin="1"/>
+<wire x1="5.08" y1="96.52" x2="5.08" y2="93.98" width="0.1524" layer="91"/>
+<pinref part="SUPPLY2" gate="G$1" pin="+9V"/>
+<junction x="5.08" y="96.52"/>
+<pinref part="R3" gate="G$1" pin="2"/>
+<wire x1="5.08" y1="96.52" x2="-7.62" y2="96.52" width="0.1524" layer="91"/>
+<pinref part="U$1" gate="G$1" pin="VIN"/>
+<label x="0" y="104.14" size="1.778" layer="95"/>
+</segment>
+<segment>
+<wire x1="182.88" y1="58.42" x2="170.18" y2="58.42" width="0.1524" layer="91"/>
+<pinref part="SW1" gate="G$1" pin="NO_2"/>
+<wire x1="165.1" y1="52.07" x2="170.18" y2="52.07" width="0.1524" layer="91"/>
+<wire x1="170.18" y1="52.07" x2="170.18" y2="58.42" width="0.1524" layer="91"/>
+<pinref part="SW1" gate="G$1" pin="NO_1"/>
+<wire x1="170.18" y1="58.42" x2="165.1" y2="58.42" width="0.1524" layer="91"/>
+<junction x="170.18" y="58.42"/>
+<label x="175.26" y="60.96" size="1.778" layer="95"/>
+</segment>
+</net>
